Commit message: return to the pos calculate of wheels for it's better used in isaac, and add friction to urdf. Add terrain more complex (not just only the stairs)

File: resources/diablo_pluspro_stand/urdf/diablo_pluspro_stand.urdf (robot description, URDF)
Before this commit: robot diablo_pluspro_stand, 7 links, 6 joints
Joints:
- joint left_wheel_joint: limit effort=20 velocity=30 -> lower=-1000000 upper=1000000 effort=20 velocity=30
- joint right_wheel_joint: limit effort=20 velocity=30 -> lower=-1000000 upper=1000000 effort=20 velocity=30

Commit message: add randomize damping, friction, armature, inertia

File: resources/diablo_pluspro_stand/urdf/diablo_pluspro_stand.urdf (robot description, URDF)
Before this commit: robot diablo_pluspro_stand, 7 links, 6 joints
Links:
- link base_link: mass 8.53 -> 11.47
- link left_knee_link: mass 2.17 -> 0.42
- link left_wheel_link: mass 2 -> 2.785
- link right_knee_link: mass 2.17 -> 0.42
- link right_wheel_link: mass 2 -> 2.785
Joints:
- joint left_knee_joint: limit lower=-1.57 upper=0 effort=80 velocity=15 -> lower=-1.19 upper=0 effort=80 velocity=15
- joint right_knee_joint: limit lower=-1.57 upper=0 effort=80 velocity=15 -> lower=-1.19 upper=0 effort=80 velocity=15
