Commit message: Add diablo_pluspro new urdf with brand new com and inertia

File: resources/diablo_pluspro/urdf/diablo_pluspro.urdf (robot description, URDF)
Before this commit: robot diablo_pluspro_stand, 7 links, 6 joints
Joints:
- joint left_hip_joint: origin xyz=0 0.14844 0.0547374 rpy=0 0 0 -> xyz=0 0.14844 0 rpy=0 0 0
- joint left_knee_joint: origin xyz=-0.124016 0 -0.156908 rpy=0 0 0 -> xyz=-0.12022 0 -0.15983 rpy=0 0 0
- joint left_wheel_joint: origin xyz=0.133344 0 -0.149062 rpy=0 0 0 -> xyz=0.13397 0 -0.1485 rpy=0 0 0
- joint right_hip_joint: origin xyz=0 -0.14844 0.0547374 rpy=0 0 0 -> xyz=0 -0.1484 0 rpy=0 0 0
- joint right_knee_joint: origin xyz=-0.124016 0 -0.156908 rpy=0 0 0 -> xyz=-0.12022 0 -0.15983 rpy=0 0 0
- joint right_wheel_joint: origin xyz=0.133344 0 -0.149062 rpy=0 0 0 -> xyz=0.13397 0 -0.1485 rpy=0 0 0
